File: PCB/PCB.kicad_sch (KiCad schematic)
At the start: 20 parts, among them J1 USB_C_Receptacle_USB2.0_14P, J2 OLED_128x64, SW1 SW_Push, U1 STM32F072CBTx, U2 USBLC6-2SC6, U3 XC6206, U5 TRRS

Commit message: Started trying to route the traces
Parts:
- C1, C2, C3, C4, C5, C6, C7: footprint (none) -> Capacitor_SMD:C_0805_2012Metric
- C8, C9: value C -> 1uF; footprint (none) -> Capacitor_SMD:C_0805_2012Metric
- F1: footprint (none) -> Fuse:Fuse_0805_2012Metric
- J1: footprint (none) -> Connector_USB:USB_C_Receptacle_HRO_TYPE-C-31-M-12
- J2: footprint ScottoKeebs_Components:OLED_128x64 -> Connector_PinHeader_2.54mm:PinHeader_1x04_P2.54mm_Vertical
- R1, R2: renamed from 5.1k; value Resistor -> 5.1k; footprint (none) -> Resistor_SMD:R_0805_2012Metric
- R3: renamed from 10k; value Resistor -> 10k; footprint (none) -> Resistor_SMD:R_0805_2012Metric
- SW1: footprint (none) -> Button_Switch_SMD:SW_SPST_TL3342
- U5: footprint ScottoKeebs_Components:TRRS_PJ-320A -> Connector_Audio:Jack_3.5mm_PJ311_Horizontal
Changed lines of the file:
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@@
 		)
 		(property "Value" "100nF"
-			(at 53.594 169.418 90)
+			(at 58.928 160.274 0)
 			(show_name no)
 			(do_not_autoplace no)
@@
 					(size 1.27 1.27)
 				)
-				(justify left)
+				(justify right)
 			)
 		)
-		(property "Footprint" ""
+		(property "Footprint" "Capacitor_SMD:C_0805_2012Metric"
 			(at 58.1152 170.18 0)
 			(hide yes)
@@
 		(in_pos_files yes)
 		(dnp no)
-		(property "Reference" "5.1k"
+		(property "Reference" "R1"
 			(at 224.79 44.45 0)
 			(show_name no)
@@
 			)
 		)
-		(property "Value" "Resistor"
+		(property "Value" "5.1k"
 			(at 224.536 42.418 0)
 			(show_name no)
@@
 			)
 		)
-		(property "Footprint" ""
+		(property "Footprint" "Resistor_SMD:R_0805_2012Metric"
 			(at 224.79 46.228 0)
 			(hide yes)
@@
 			(project "PCB"
 				(path "/61897acb-2078-4c47-92ce-82a0439bac7e"
-					(reference "5.1k")
+					(reference "R1")
 					(unit 1)
 				)
@@
 			)
 		)
-		(property "Footprint" "ScottoKeebs_Components:TRRS_PJ-320A"
+		(property "Footprint" "Connector_Audio:Jack_3.5mm_PJ311_Horizontal"
 			(at 154.94 81.28 0)
 			(hide yes)
@@
 		)
 		(property "Value" "100nF"
-			(at 43.434 169.418 90)
+			(at 48.514 160.528 0)
 			(show_name no)
 			(do_not_autoplace no)
@@
 					(size 1.27 1.27)
 				)
-				(justify left)
+				(justify right)
 			)
 		)
-		(property "Footprint" ""
+		(property "Footprint" "Capacitor_SMD:C_0805_2012Metric"
 			(at 47.9552 170.18 0)
 			(hide yes)
@@
 		)
 		(property "Value" "10nF"
-			(at 73.914 169.418 90)
+			(at 74.676 161.036 0)
 			(show_name no)
 			(do_not_autoplace no)
@@
 			)
 		)
-		(property "Footprint" ""
+		(property "Footprint" "Capacitor_SMD:C_0805_2012Metric"
 			(at 78.4352 170.18 0)
 			(hide yes)
@@
 		)
 		(property "Value" "100nF"
-			(at 23.114 169.418 90)
+			(at 22.606 168.148 90)
 			(show_name no)
 			(do_not_autoplace no)
@@
 			)
 		)
-		(property "Footprint" ""
+		(property "Footprint" "Capacitor_SMD:C_0805_2012Metric"
 			(at 27.6352 170.18 0)
 			(hide yes)
@@
 			)
 		)
-		(property "Footprint" ""
+		(property "Footprint" "Fuse:Fuse_0805_2012Metric"
 			(at 229.87 41.148 0)
 			(hide yes)
@@
 			)
 		)
-		(property "Value" "C"
+		(property "Value" "1uF"
 			(at 254 40.6399 0)
 			(show_name no)
@@
 			)
 		)
-		(property "Footprint" ""
+		(property "Footprint" "Capacitor_SMD:C_0805_2012Metric"
 			(at 251.1552 43.18 0)
 			(hide yes)
@@
 		)
 		(property "Value" "100nF"
-			(at 33.274 169.418 90)
+			(at 38.862 160.274 0)
 			(show_name no)
 			(do_not_autoplace no)
@@
 					(size 1.27 1.27)
 				)
-				(justify left)
+				(justify right)
 			)
 		)
-		(property "Footprint" ""
+		(property "Footprint" "Capacitor_SMD:C_0805_2012Metric"
 			(at 37.7952 170.18 0)
 			(hide yes)
@@
 		(in_pos_files yes)
 		(dnp no)
-		(property "Reference" "5.1k"
+		(property "Reference" "R2"
 			(at 224.79 46.99 0)
 			(show_name no)
@@
 			)
 		)
-		(property "Value" "Resistor"
+		(property "Value" "5.1k"
 			(at 225.298 49.276 0)
 			(show_name no)
@@
 			)
 		)
-		(property "Footprint" ""
+		(property "Footprint" "Resistor_SMD:R_0805_2012Metric"
 			(at 224.79 48.768 0)
 			(hide yes)
@@
 			(project "PCB"
 				(path "/61897acb-2078-4c47-92ce-82a0439bac7e"
-					(reference "5.1k")
+					(reference "R2")
 					(unit 1)
 				)
@@
 			)
 		)
-		(property "Footprint" "ScottoKeebs_Components:OLED_128x64"
+		(property "Footprint" "Connector_PinHeader_2.54mm:PinHeader_1x04_P2.54mm_Vertical"
 			(at 92.71 82.55 0)
 			(hide yes)
@@
 			)
 		)
-		(property "Footprint" ""
+		(property "Footprint" "Connector_USB:USB_C_Receptacle_HRO_TYPE-C-31-M-12"
 			(at 208.28 54.61 0)
 			(hide yes)
@@
 			)
 		)
-		(property "Footprint" ""
+		(property "Footprint" "Button_Switch_SMD:SW_SPST_TL3342"
 			(at 91.44 97.79 0)
 			(hide yes)
@@
 			)
 		)
-		(property "Footprint" ""
+		(property "Footprint" "Capacitor_SMD:C_0805_2012Metric"
 			(at 30.48 63.8048 0)
 			(hide yes)
@@
 		(in_pos_files yes)
 		(dnp no)
-		(fields_autoplaced yes)
-		(property "Reference" "10k"
-			(at 104.14 96.52 0)
+		(property "Reference" "R3"
+			(at 104.14 102.87 0)
 			(show_name no)
 			(do_not_autoplace no)
@@
 			)
 		)
-		(property "Value" "Resistor"
-			(at 104.14 99.06 0)
+		(property "Value" "10k"
+			(at 103.886 100.33 0)
 			(show_name no)
 			(do_not_autoplace no)
@@
 			)
 		)
-		(property "Footprint" ""
+		(property "Footprint" "Resistor_SMD:R_0805_2012Metric"
 			(at 104.14 104.648 0)
 			(hide yes)
@@
 			(project "PCB"
 				(path "/61897acb-2078-4c47-92ce-82a0439bac7e"
-					(reference "10k")
+					(reference "R3")
 					(unit 1)
 				)
@@
 			)
 		)
-		(property "Value" "C"
+		(property "Value" "1uF"
 			(at 275.59 40.6399 0)
 			(show_name no)
@@
 			)
 		)
-		(property "Footprint" ""
+		(property "Footprint" "Capacitor_SMD:C_0805_2012Metric"
 			(at 272.7452 43.18 0)
 			(hide yes)
@@
 		)
 		(property "Value" "100nF"
-			(at 63.754 169.418 90)
+			(at 65.024 161.036 0)
 			(show_name no)
 			(do_not_autoplace no)
@@
 			)
 		)
-		(property "Footprint" ""
+		(property "Footprint" "Capacitor_SMD:C_0805_2012Metric"
 			(at 68.2752 170.18 0)
 			(hide yes)
